File: hardware/usb_8285_tiny/usb_8285_tiny.kicad_pcb (KiCad board)
At the start: 2 copper layers, 12.7 x 12 mm, 23 parts, among them M1 5.6p, M2 5.6p, M3 5.6p, P1 UTX, P10 ADC, P2 URX, P3 D+, P4 +5V, P5 +5V, P6 GND, P7 GND, P8 D-, P9 G0, U1 8285, U2 1824, X1 26M

Commit message: add tiny
Parts:
- M3: footprint SM0402 -> SM0603
- moved C4 0.83 mm to (49.6, 29.4)
- moved M3 0.34 mm to (49.3, 31.3)
- moved A1 0.13 mm to (47.2, 32.0)
- moved P10 0.08 mm to (50.4, 33.2)
Routing:
- net GND: track 61.0 -> 84.7 mm, vias 5 -> 7
- net +3.3V: track 71.6 -> 53.8 mm, vias 5 -> 3
