File: hardware/usb_8285_tiny/usb_8285_tiny.sch (KiCad schematic (older format))
At the start: 23 parts, among them M1 5.6p, M2 5.6p, M3 5.6p, P1 UTX, P10 ADC, P2 URX, P3 D+, P4 +5V, P5 +5V, P6 GND, P7 GND, P8 D-, P9 G0, U1 8285, U2 1824, X1 26M

Commit message: add tiny
Parts:
- M3: footprint SM0402 -> SM0603
Changed lines of the file:
@@
 F 0 "M3" H 3050 2250 40  0000 L CNN
 F 1 "5.6p" H 3056 2065 40  0000 L CNN
-F 2 "SM0402" H 3088 2000 30  0000 C CNN
+F 2 "SM0603" H 3088 2000 30  0000 C CNN
 F 3 "~" H 3050 2150 60  0000 C CNN
 	1    3050 2150
